Commit message: add support for arm and camera

File: urdf/my_robot.urdf.xacro (robot description, xacro)
@@ -3,3 +3,11 @@
     <xacro:include filename="common_properties.xacro" />
     <xacro:include filename="mobile_base.xacro" />
+    <xacro:include filename="mobile_base_gazebo.xacro" />
+    <xacro:include filename="arm.xacro" />
+    <xacro:include filename="camera.xacro" />
+    <joint name="mobile_base_arm_joint" type="fixed">
+        <parent link="base_link" />
+        <child link="arm_base_link" />
+        <origin xyz="${(base_length + arm_length) / 4.0} 0 ${base_height}" rpy="0 0 0" />
+    </joint>
 </robot>

File: urdf/smart_base.xacro (robot description, xacro)
@@ -26,5 +26,5 @@
             xyz="0 0 ${base_height / 2.0}" rpy="0 0 0" />
     </link>
-    <xacro:macro name="wheel_link" params="prefix">
+        <xacro:macro name="wheel_link" params="prefix">
         <link name="${prefix}_wheel_link">
             <visual>
@@ -86,3 +86,41 @@
         <axis xyz="0 1 0" />
     </joint>
+    <gazebo reference="base_link">
+        <material> Gazebo/Blue </material>
+    </gazebo>
+    <gazebo reference="right_wheel_link">
+        <material> Gazebo/Grey</material>
+    </gazebo>
+    <gazebo reference="left_wheel_link">
+        <material> Gazebo/Grey</material>
+    </gazebo>
+    <gazebo reference="castor_wheel_link">
+        <material> Gazebo/Grey</material>
+        <mu1 value="0.1"/>
+        <mu2 value="0.1"/>
+    </gazebo>
+      <gazebo>
+    <!-- taken from
+     https://raw.githubusercontent.com/ros-simulation/gazebo_ros_pkgs/refs/heads/ros2/gazebo_plugins/include/gazebo_plugins/gazebo_ros_diff_drive.hpp
+    -->
+        <plugin name="diff_drive_controller" filename="libgazebo_ros_diff_drive.so">
+            <!-- Update rate in Hz -->
+            <update_rate>50</update_rate>
+            <!-- wheels -->
+            <left_joint>base_left_wheel_joint</left_joint>
+            <right_joint>base_right_wheel_joint</right_joint>
+            <!-- kinematics -->
+            <wheel_separation>0.45</wheel_separation> <!-- dstince 0.4 + 0.5 base_width + length of cyclnder-->
+            <wheel_diameter>0.2</wheel_diameter> <!-- wheel_radius * 2-->
+            <!-- input -->
+            <command_topic>cmd_vel</command_topic>
+            <!-- output -->
+            <publish_odom>true</publish_odom> <!-- odementry to know where the robot is relative to the origin-->
+            <publish_odom_tf>true</publish_odom_tf>
+            <publish_wheel_tf>true</publish_wheel_tf>
+            <odometry_topic>odom</odometry_topic>
+            <odometry_frame>odom</odometry_frame>
+            <robot_base_frame>base_footprint</robot_base_frame> <!-- root frame of the robot, aka the base_footprint link-->
+        </plugin>
+    </gazebo>
 </robot>

File: urdf/smart_common_properties.xacro (robot description, xacro)
@@ -16,8 +16,5 @@
         <color rgba="0.5 0.5 0.5 1" />
     </material>
-    <!-- https://en.wikipedia.org/wiki/List_of_moments_of_inertia#List_of_3D_inertia_tensors-->
-    <!--
-    https://docs.ros.org/en/jazzy/Tutorials/Intermediate/URDF/Adding-Physical-and-Collision-Properties-to-a-URDF-Model.html-->
-    <xacro:macro name="box_inertia"
+        <xacro:macro name="box_inertia"
         params="m l w h xyz rpy">
         <inertial>
